File: reference_circuit.kicad_sch (KiCad schematic)
At the start: 14 parts, among them U11 OPA4202, U2 LM399

Commit message: Updated references to follow geographical rules
Parts:
- renumbered C55 to C59, C44 to C65, C56 to C71, C58 to C89, C57 to C90, L11 to L19, NT3 to NT21, R52 to R55, R53 to R56, R55 to R61, R54 to R62, R51 to R9, U2 to U12, U11 to U24

Commit message: Fixed footprints
Parts:
- R5: renamed from R9; footprint Capacitor_SMD:C_0805_2012Metric -> Resistor_SMD:R_0805_2012Metric
- R50: renamed from R55; footprint Capacitor_SMD:C_0603_1608Metric -> Resistor_SMD:R_0603_1608Metric
- renumbered C71 to C47, C65 to C52, C59 to C57, C90 to C7, C89 to C8, L19 to L4, NT21 to NT5, R62 to R39, R61 to R40, R56 to R46, U24 to U22, U12 to U7
Connections:
- net at R46.1: now also U22.3 (+); no longer U22.10 (+)
- net at C47.1, R39.2: now also U22.1; no longer U22.8
- net at C47.2, R40.2: now also U22.2 (-); no longer U22.9 (-)
Changed lines of the file:
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@@
 		(on_board yes)
 		(dnp no)
-		(property "Reference" "R9"
+		(property "Reference" "R5"
 			(at 93.98 68.58 0)
 			(effects
@@
 			)
 		)
-		(property "Footprint" "Capacitor_SMD:C_0805_2012Metric"
+		(property "Footprint" "Resistor_SMD:R_0805_2012Metric"
 			(at 89.662 69.85 90)
 			(effects
@@
 		(on_board yes)
 		(dnp no)
-		(property "Reference" "R55"
+		(property "Reference" "R50"
 			(at 113.03 78.74 0)
 			(effects
@@
 			)
 		)
-		(property "Footprint" "Capacitor_SMD:C_0603_1608Metric"
+		(property "Footprint" "Resistor_SMD:R_0603_1608Metric"
 			(at 108.712 80.01 90)
 			(effects
@@
 		(on_board yes)
 		(dnp no)
-		(property "Reference" "C59"
+		(property "Reference" "C57"
 			(at 114.3 88.9 0)
 			(effects
@@
 		(lib_id "Amplifier_Operational:OPA4197xD")
 		(at 142.24 77.47 0)
-		(unit 3)
+		(unit 1)
 		(exclude_from_sim no)
 		(in_bom yes)
 		(on_board yes)
 		(dnp no)
-		(property "Reference" "U24"
+		(property "Reference" "U22"
 			(at 142.24 67.31 0)
 			(effects
@@
 		(on_board yes)
 		(dnp no)
-		(property "Reference" "L19"
+		(property "Reference" "L4"
 			(at 207.01 74.93 0)
 			(effects
@@
 		(on_board yes)
 		(dnp no)
-		(property "Reference" "C90"
+		(property "Reference" "C7"
 			(at 191.77 81.28 0)
 			(effects
@@
 		(on_board yes)
 		(dnp no)
-		(property "Reference" "U12"
+		(property "Reference" "U7"
 			(at 93.98 82.55 0)
 			(effects
@@
 		(on_board yes)
 		(dnp no)
-		(property "Reference" "R62"
+		(property "Reference" "R39"
 			(at 166.37 71.12 90)
 			(effects
@@
 		(on_board yes)
 		(dnp no)
-		(property "Reference" "R61"
+		(property "Reference" "R40"
 			(at 166.37 92.71 90)
 			(effects
@@
 		(on_board yes)
 		(dnp no)
-		(property "Reference" "C71"
+		(property "Reference" "C47"
 			(at 158.75 86.36 0)
 			(effects
@@
 		(on_board yes)
 		(dnp no)
-		(property "Reference" "C65"
+		(property "Reference" "C52"
 			(at 78.74 83.82 0)
 			(effects
@@
 		(on_board yes)
 		(dnp no)
-		(property "Reference" "C89"
+		(property "Reference" "C8"
 			(at 229.87 81.28 0)
 			(effects
@@
 		(on_board yes)
 		(dnp no)
-		(property "Reference" "R56"
+		(property "Reference" "R46"
 			(at 124.46 68.58 90)
 			(effects
@@
 		(on_board yes)
 		(dnp no)
-		(property "Reference" "NT21"
+		(property "Reference" "NT5"
 			(at 119.38 99.06 0)
 			(effects
