File: reference_circuit.kicad_sch (KiCad schematic)
At the start: 14 parts, among them U11 OPA4202, U2 LM399

Commit message: Update references (#5)
* Updated references to follow geographical rules

* Updated stackup
Parts:
- R5: renamed from R51; footprint Capacitor_SMD:C_0805_2012Metric -> Resistor_SMD:R_0805_2012Metric
- R50: renamed from R52; footprint Capacitor_SMD:C_0603_1608Metric -> Resistor_SMD:R_0603_1608Metric
- renumbered C56 to C47, C44 to C52, C55 to C57, C57 to C7, C58 to C8, L11 to L4, NT3 to NT5, R54 to R39, R55 to R40, R53 to R46, U11 to U22, U2 to U7
Connections:
- net at R46.1: now also U22.3 (+); no longer U22.10 (+)
- net at C47.1, R39.2: now also U22.1; no longer U22.8
- net at C47.2, R40.2: now also U22.2 (-); no longer U22.9 (-)

Commit message: Added RoHS info
Parts:
- C59: renamed from C57; RoHS (none) -> Yes; Temperature (none) -> Tstorage = –55 °C to 155 °C
- C65: renamed from C52; RoHS (none) -> Yes; Temperature (none) -> Tstorage = –55 °C to 155 °C
- C71: renamed from C47; RoHS (none) -> Yes; Temperature (none) -> Tstorage = –55 °C to 155 °C
- C89: renamed from C8; RoHS (none) -> Yes; Temperature (none) -> Tstorage = –55 °C to 155 °C
- C90: renamed from C7; RoHS (none) -> Yes; Temperature (none) -> Tstorage = –55 °C to 155 °C
- L19: renamed from L4; RoHS (none) -> Yes; Temperature (none) -> Tstorage = –40 °C to 125 °C
- R55: renamed from R50; RoHS (none) -> By exemption; Temperature (none) -> Tstorage = –55 °C to 155 °C
- R56: renamed from R46; RoHS (none) -> Yes; Temperature (none) -> Tstorage = –55 °C to 125 °C
- R61: renamed from R40; RoHS (none) -> Yes; Temperature (none) -> Tstorage = –55 °C to 125 °C
- R62: renamed from R39; RoHS (none) -> Yes; Temperature (none) -> Tstorage = –55 °C to 125 °C
- R9: renamed from R5; RoHS (none) -> Yes; Temperature (none) -> Tstorage = –55 °C to 125 °C
- U12: renamed from U7; RoHS (none) -> Yes; Temperature (none) -> Tstorage = –55 °C to 105 °C
- U24: renamed from U22; RoHS (none) -> Yes; Temperature (none) -> Tstorage = –40 °C to 125 °C
- renumbered NT5 to NT21
Connections:
- net at C71.1, R62.2: now also U24.8; no longer U24.1
- net at C71.2, R61.2: now also U24.9 (-); no longer U24.2 (-)
- net at R56.1: now also U24.10 (+); no longer U24.3 (+)

Commit message: Bump version to 1.0.2
Parts:
- renumbered C71 to C47, C65 to C52, C59 to C57, C90 to C7, C89 to C8, L19 to L4, NT21 to NT5, R62 to R39, R61 to R40, R56 to R46, R9 to R5, R55 to R50, U24 to U22, U12 to U7
Connections:
- net at R46.1: now also U22.3 (+); no longer U22.10 (+)
- net at C47.1, R39.2: now also U22.1; no longer U22.8
- net at C47.2, R40.2: now also U22.2 (-); no longer U22.9 (-)
Changed lines of the file:
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@@
 		(title "LM399/ADR1399 Burnin Board")
 		(date "2024-11-21")
-		(rev "1.0.1")
+		(rev "1.0.2")
 		(company "TU Darmstadt, IAP, APQ")
 		(comment 1 "Copyright (©) 2021, Patrick Baus <patrick.baus@physik.tu-darmstadt.de>")
@@
 		(on_board yes)
 		(dnp no)
-		(property "Reference" "R9"
+		(property "Reference" "R5"
 			(at 93.98 68.58 0)
 			(effects
@@
 		(on_board yes)
 		(dnp no)
-		(property "Reference" "R55"
+		(property "Reference" "R50"
 			(at 113.03 78.74 0)
 			(effects
@@
 		(on_board yes)
 		(dnp no)
-		(property "Reference" "C59"
+		(property "Reference" "C57"
 			(at 114.3 88.9 0)
 			(effects
@@
 		(lib_id "Amplifier_Operational:OPA4197xD")
 		(at 142.24 77.47 0)
-		(unit 3)
+		(unit 1)
 		(exclude_from_sim no)
 		(in_bom yes)
 		(on_board yes)
 		(dnp no)
-		(property "Reference" "U24"
+		(property "Reference" "U22"
 			(at 142.24 67.31 0)
 			(effects
@@
 		(on_board yes)
 		(dnp no)
-		(property "Reference" "L19"
+		(property "Reference" "L4"
 			(at 207.01 74.93 0)
 			(effects
@@
 		(on_board yes)
 		(dnp no)
-		(property "Reference" "C90"
+		(property "Reference" "C7"
 			(at 191.77 81.28 0)
 			(effects
@@
 		(on_board yes)
 		(dnp no)
-		(property "Reference" "U12"
+		(property "Reference" "U7"
 			(at 93.98 82.55 0)
 			(effects
@@
 		(on_board yes)
 		(dnp no)
-		(property "Reference" "R62"
+		(property "Reference" "R39"
 			(at 166.37 71.12 90)
 			(effects
@@
 		(on_board yes)
 		(dnp no)
-		(property "Reference" "R61"
+		(property "Reference" "R40"
 			(at 166.37 92.71 90)
 			(effects
@@
 		(on_board yes)
 		(dnp no)
-		(property "Reference" "C71"
+		(property "Reference" "C47"
 			(at 158.75 86.36 0)
 			(effects
@@
 		(on_board yes)
 		(dnp no)
-		(property "Reference" "C65"
+		(property "Reference" "C52"
 			(at 78.74 83.82 0)
 			(effects
@@
 		(on_board yes)
 		(dnp no)
-		(property "Reference" "C89"
+		(property "Reference" "C8"
 			(at 229.87 81.28 0)
 			(effects
@@
 		(on_board yes)
 		(dnp no)
-		(property "Reference" "R56"
+		(property "Reference" "R46"
 			(at 124.46 68.58 90)
 			(effects
@@
 		(on_board yes)
 		(dnp no)
-		(property "Reference" "NT21"
+		(property "Reference" "NT5"
 			(at 119.38 99.06 0)
 			(effects
