File: lm399_burnin_board.kicad_pcb (KiCad board)
At the start: 4 copper layers, 160 x 100 mm, 287 parts, among them J1 DB50_Female, J2 C64AC, U1 LM399, U10 LM399, U11 LM399, U12 LM399, U13 LM399, U14 LM399, U15 LM399, U16 LM399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

Commit message: Updated stackup
Parts:
- R1, R10, R11, R12, R13, R14, R17, R18, R2, R3, R31, R36, R4, R5, R6, R69, R7, R8, R9, R92: footprint Capacitor_SMD:C_0805_2012Metric -> Resistor_SMD:R_0805_2012Metric
- R101, R102, R19, R20, R21, R22, R49, R50, R51, R52, R53, R54, R55, R59, R82, R83, R84, R85, R86, R87: footprint Capacitor_SMD:C_0603_1608Metric -> Resistor_SMD:R_0603_1608Metric
Connections:
- net /sheet61977749/GND_heater renamed /Reference Block 2/GND_heater
- net /sheet61977749/GND_zener renamed /Reference Block 2/GND_zener
- net /sheet61977B89/GND_heater renamed /Reference Block 3/GND_heater
- net /sheet61977B89/GND_zener renamed /Reference Block 3/GND_zener
- net /sheet6197811F/GND_heater renamed /Reference Block 4/GND_heater
- net /sheet6197811F/GND_zener renamed /Reference Block 4/GND_zener
- net /sheet6197BEAD/GND_heater renamed /Reference Block 5/GND_heater
- net /sheet6197BEAD/GND_zener renamed /Reference Block 5/GND_zener
Other:
- board text added: "0.196 mm"
- board text added: "0.203 mm"
- board text added: "1.03 mm"
- board text added: "Prepreg 7628"
- board text added: "Prepreq 7628"
- board text removed: "0.1 mm"
- board text removed: "0.11 mm"
- board text removed: "1.13 mm"
- board text removed: "1.265 mm"
- board text removed: "Prepreg 2313"
- board text removed: "Prepreq 2313"
