File: lm399_burnin_board.kicad_pcb (KiCad board)
At the start: 4 copper layers, 160 x 100 mm, 287 parts, among them J1 C64AC, J2 DB50_Female, U1 OPA4202, U10 LM399, U11 OPA4202, U12 LM399, U13 LM399, U14 LM399, U15 LM399, U16 OPA4202, U17 LM399, U18 LM399, U19 LM399, U2 LM399, U20 LM399, U21 OPA4202, U22 LM399, U23 LM399, U24 LM399, U25 LM399, U26 LT1085-ADJ, U3 LM399, U4 LM399, U5 LM399, U6 OPA4202, U7 LM399, U8 LM399, U9 LM399

Commit message: Update references (#5)
* Updated references to follow geographical rules

* Updated stackup
Parts:
- R1: renamed from R91; footprint Capacitor_SMD:C_0805_2012Metric -> Resistor_SMD:R_0805_2012Metric
- R10: renamed from R21; footprint Capacitor_SMD:C_0805_2012Metric -> Resistor_SMD:R_0805_2012Metric
- R101: renamed from R77; footprint Capacitor_SMD:C_0603_1608Metric -> Resistor_SMD:R_0603_1608Metric
- R102: renamed from R62; footprint Capacitor_SMD:C_0603_1608Metric -> Resistor_SMD:R_0603_1608Metric
- R11: renamed from R36; footprint Capacitor_SMD:C_0805_2012Metric -> Resistor_SMD:R_0805_2012Metric
- R12: renamed from R41; footprint Capacitor_SMD:C_0805_2012Metric -> Resistor_SMD:R_0805_2012Metric
- R13: renamed from R56; footprint Capacitor_SMD:C_0805_2012Metric -> Resistor_SMD:R_0805_2012Metric
- R14: renamed from R71; footprint Capacitor_SMD:C_0805_2012Metric -> Resistor_SMD:R_0805_2012Metric
- R17: renamed from R61; footprint Capacitor_SMD:C_0805_2012Metric -> Resistor_SMD:R_0805_2012Metric
- R18: renamed from R76; footprint Capacitor_SMD:C_0805_2012Metric -> Resistor_SMD:R_0805_2012Metric
- R19: renamed from R12; footprint Capacitor_SMD:C_0603_1608Metric -> Resistor_SMD:R_0603_1608Metric
- R2: renamed from R11; footprint Capacitor_SMD:C_0805_2012Metric -> Resistor_SMD:R_0805_2012Metric
- R20: renamed from R7; footprint Capacitor_SMD:C_0603_1608Metric -> Resistor_SMD:R_0603_1608Metric
- R21: renamed from R92; footprint Capacitor_SMD:C_0603_1608Metric -> Resistor_SMD:R_0603_1608Metric
- R22: renamed from R87; footprint Capacitor_SMD:C_0603_1608Metric -> Resistor_SMD:R_0603_1608Metric
- R3: renamed from R81; footprint Capacitor_SMD:C_0805_2012Metric -> Resistor_SMD:R_0805_2012Metric
- R31: renamed from R6; footprint Capacitor_SMD:C_0805_2012Metric -> Resistor_SMD:R_0805_2012Metric
- R36: renamed from R86; footprint Capacitor_SMD:C_0805_2012Metric -> Resistor_SMD:R_0805_2012Metric
- R4: renamed from R96; footprint Capacitor_SMD:C_0805_2012Metric -> Resistor_SMD:R_0805_2012Metric
- R49: renamed from R17; footprint Capacitor_SMD:C_0603_1608Metric -> Resistor_SMD:R_0603_1608Metric
- R5: renamed from R1; footprint Capacitor_SMD:C_0805_2012Metric -> Resistor_SMD:R_0805_2012Metric
- R50: renamed from R2; footprint Capacitor_SMD:C_0603_1608Metric -> Resistor_SMD:R_0603_1608Metric
- R51: renamed from R97; footprint Capacitor_SMD:C_0603_1608Metric -> Resistor_SMD:R_0603_1608Metric
- R52: renamed from R82; footprint Capacitor_SMD:C_0603_1608Metric -> Resistor_SMD:R_0603_1608Metric
- R53: renamed from R47; footprint Capacitor_SMD:C_0603_1608Metric -> Resistor_SMD:R_0603_1608Metric
- R54: renamed from R27; footprint Capacitor_SMD:C_0603_1608Metric -> Resistor_SMD:R_0603_1608Metric
- R55: renamed from R52; footprint Capacitor_SMD:C_0603_1608Metric -> Resistor_SMD:R_0603_1608Metric
- R59: renamed from R32; footprint Capacitor_SMD:C_0603_1608Metric -> Resistor_SMD:R_0603_1608Metric
- R6: renamed from R16; footprint Capacitor_SMD:C_0805_2012Metric -> Resistor_SMD:R_0805_2012Metric
- R69: renamed from R26; footprint Capacitor_SMD:C_0805_2012Metric -> Resistor_SMD:R_0805_2012Metric
- R7: renamed from R31; footprint Capacitor_SMD:C_0805_2012Metric -> Resistor_SMD:R_0805_2012Metric
- R8: renamed from R46; footprint Capacitor_SMD:C_0805_2012Metric -> Resistor_SMD:R_0805_2012Metric
- R82: renamed from R57; footprint Capacitor_SMD:C_0603_1608Metric -> Resistor_SMD:R_0603_1608Metric
- R83: renamed from R42; footprint Capacitor_SMD:C_0603_1608Metric -> Resistor_SMD:R_0603_1608Metric
- R84: renamed from R37; footprint Capacitor_SMD:C_0603_1608Metric -> Resistor_SMD:R_0603_1608Metric
- R85: renamed from R22; footprint Capacitor_SMD:C_0603_1608Metric -> Resistor_SMD:R_0603_1608Metric
- R86: renamed from R67; footprint Capacitor_SMD:C_0603_1608Metric -> Resistor_SMD:R_0603_1608Metric
- R87: renamed from R72; footprint Capacitor_SMD:C_0603_1608Metric -> Resistor_SMD:R_0603_1608Metric
- R9: renamed from R51; footprint Capacitor_SMD:C_0805_2012Metric -> Resistor_SMD:R_0805_2012Metric
- R92: renamed from R66; footprint Capacitor_SMD:C_0805_2012Metric -> Resistor_SMD:R_0805_2012Metric
- renumbered C94 to C1, C105 to C10, C72 to C100, C82 to C101, C67 to C102, C64 to C103, C70 to C104, C81 to C105, C75 to C106, C66 to C107, C89 to C11, C90 to C12, C31 to C13, C32 to C14, C62 to C15, C63 to C16, C47 to C17, C48 to C18, C41 to C19, C95 to C2, C42 to C20, C26 to C21, C27 to C22, C73 to C23, C74 to C24, C106 to C25, C107 to C26, C83 to C27, C84 to C28, C68 to C29, C10 to C3, C69 to C30, C12 to C31, C13 to C32, C7 to C33, C8 to C34, C86 to C35, C97 to C36, C101 to C37, C92 to C38, C14 to C39, C11 to C4, C9 to C40, C1 to C41, C98 to C42, C85 to C43, C93 to C44, C17 to C45, C19 to C46, C4 to C47, C91 to C48, C103 to C49, C20 to C5, C88 to C50, C18 to C51, C2 to C52, C102 to C53, C96 to C54, C100 to C55, C99 to C56, C3 to C57, C87 to C58, C55 to C59, C21 to C6, C50 to C60, C34 to C61, C29 to C62, C16 to C63, C15 to C64, C44 to C65, C59 to C66, C23 to C67, C38 to C68, C37 to C69, C5 to C7, C36 to C70, C56 to C71, C51 to C72, C35 to C73, C30 to C74, C53 to C75, C52 to C76, C61 to C77, C43 to C78, C46 to C79, C6 to C8, C40 to C80, C25 to C81, C22 to C82, C49 to C83, C60 to C84, C54 to C85, C28 to C86, C39 to C87, C33 to C88, C58 to C89, C104 to C9, C57 to C90, C45 to C91, C24 to C92, C79 to C93, C78 to C94, C76 to C95, C71 to C96, C65 to C97, C80 to C98, C77 to C99, J2 to J1, J1 to J2, L18 to L1, L8 to L10, L5 to L11, L14 to L12, L16 to L13, L13 to L14, L19 to L15, L3 to L16, L7 to L17, L10 to L18, L11 to L19, L15 to L20, L4 to L3, L1 to L4, L20 to L5, L17 to L6, L6 to L7, L12 to L8, NT10 to NT1, NT16 to NT10, NT1 to NT11, NT4 to NT12, NT6 to NT13, NT46 to NT14, NT5 to NT15, NT8 to NT16, NT19 to NT17, NT11 to NT18, NT25 to NT19, NT18 to NT2, NT23 to NT20, NT3 to NT21, NT15 to NT22, NT21 to NT23, NT7 to NT25, NT22 to NT26, NT9 to NT3, NT12 to NT4, NT17 to NT5, NT20 to NT6, NT14 to NT7, NT2 to NT8, NT13 to NT9, R63 to R100, R102 to R15, R101 to R16, R13 to R23, R8 to R24, R93 to R25, R88 to R26, R14 to R27, R15 to R28, R9 to R29, R10 to R30, R95 to R32, R94 to R33, R90 to R34, R89 to R35, R19 to R37, R20 to R38, R4 to R39, R5 to R40, R99 to R41, R100 to R42, R84 to R43, R85 to R44, R18 to R45, R3 to R46, R98 to R47, R83 to R48, R53 to R56, R48 to R57, R33 to R58, R28 to R60, R55 to R61, R54 to R62, R50 to R63, R49 to R64, R35 to R65, R34 to R66, R29 to R67, R30 to R68, R59 to R70, R60 to R71, R45 to R72, R44 to R73, R39 to R74, R40 to R75, R25 to R76, R24 to R77, R58 to R78, R43 to R79, R38 to R80, R23 to R81, R73 to R88, R68 to R89, R74 to R90, R69 to R91, R75 to R93, R79 to R94, R80 to R95, R65 to R96, R70 to R97, R64 to R98, R78 to R99, U23 to U1, U9 to U10, U13 to U11, U14 to U12, U7 to U13, U10 to U14, U12 to U15, U15 to U16, U18 to U17, U19 to U18, U17 to U19, U24 to U2, U26 to U21, U1 to U22, U21 to U23, U11 to U24, U6 to U25, U16 to U26, U22 to U5, U25 to U6, U2 to U7, U5 to U8, U8 to U9
Connections:
- net /sheet61977749/GND_heater renamed /Reference Block 2/GND_heater
- net /sheet61977749/GND_zener renamed /Reference Block 2/GND_zener
- net /sheet61977B89/GND_heater renamed /Reference Block 3/GND_heater
- net /sheet61977B89/GND_zener renamed /Reference Block 3/GND_zener
- net /sheet6197811F/GND_heater renamed /Reference Block 4/GND_heater
- net /sheet6197811F/GND_zener renamed /Reference Block 4/GND_zener
- net /sheet6197BEAD/GND_heater renamed /Reference Block 5/GND_heater
- net /sheet6197BEAD/GND_zener renamed /Reference Block 5/GND_zener
Other:
- board text added: "0.196 mm"
- board text added: "0.203 mm"
- board text added: "1.03 mm"
- board text added: "Prepreg 7628"
- board text added: "Prepreq 7628"
- board text removed: "0.1 mm"
- board text removed: "0.11 mm"
- board text removed: "1.13 mm"
- board text removed: "1.265 mm"
- board text removed: "Prepreg 2313"
- board text removed: "Prepreq 2313"

Commit message: Fixed silkscreen labels
Connections:
- C31 pad 2: /Reference Block 1/GND_heater -> /Reference Block 6/GND_heater
- C32 pad 2: /Reference Block 1/GND_heater -> /Reference Block 6/GND_heater
- C33 pad 2: /Reference Block 1/GND_heater -> /Reference Block 6/GND_heater
- C34 pad 2: /Reference Block 1/GND_heater -> /Reference Block 6/GND_heater
- C35 pad 2: /Reference Block 5/GND_heater -> /Reference Block 1/GND_heater
- C36 pad 2: /Reference Block 5/GND_heater -> /Reference Block 1/GND_heater
- C37 pad 2: /Reference Block 5/GND_heater -> /Reference Block 1/GND_heater
- C38 pad 2: /Reference Block 5/GND_heater -> /Reference Block 1/GND_heater
- C45 pad 2: /Reference Block 1/GND_heater -> /Reference Block 6/GND_heater
- C48 pad 2: /Reference Block 5/GND_heater -> /Reference Block 1/GND_heater
- C51 pad 2: /Reference Block 1/GND_heater -> /Reference Block 6/GND_heater
- C52 pad 2: /Reference Block 1/GND_heater -> /Reference Block 6/GND_heater
- C53 pad 2: /Reference Block 5/GND_heater -> /Reference Block 1/GND_heater
- C54 pad 2: /Reference Block 5/GND_heater -> /Reference Block 1/GND_heater
- C57 pad 2: /Reference Block 1/GND_heater -> /Reference Block 6/GND_heater
- C58 pad 2: /Reference Block 5/GND_heater -> /Reference Block 1/GND_heater
- NT1 pad 1: /Reference Block 5/GND_zener -> /Reference Block 1/GND_zener
- NT17 pad 1: /Reference Block 1/GND_zener -> /Reference Block 6/GND_zener
- NT18 pad 1: /Reference Block 5/GND_zener -> /Reference Block 1/GND_zener
- NT19 pad 2: /Reference Block 1/GND_heater -> /Reference Block 6/GND_heater
- NT19 pad 3: /Reference Block 1/GND_zener -> /Reference Block 6/GND_zener
- NT2 pad 1: /Reference Block 1/GND_zener -> /Reference Block 6/GND_zener
- NT20 pad 2: /Reference Block 5/GND_heater -> /Reference Block 1/GND_heater
- NT20 pad 3: /Reference Block 5/GND_zener -> /Reference Block 1/GND_zener
- NT3 pad 1: /Reference Block 5/GND_zener -> /Reference Block 1/GND_zener
- NT4 pad 1: /Reference Block 5/GND_zener -> /Reference Block 1/GND_zener
- NT5 pad 1: /Reference Block 1/GND_zener -> /Reference Block 6/GND_zener
- NT6 pad 1: /Reference Block 1/GND_zener -> /Reference Block 6/GND_zener
- U1 pad 2: /Reference Block 5/GND_zener -> /Reference Block 1/GND_zener
- U1 pad 4: /Reference Block 5/GND_heater -> /Reference Block 1/GND_heater
- U2 pad 2: /Reference Block 5/GND_zener -> /Reference Block 1/GND_zener
- U2 pad 4: /Reference Block 5/GND_heater -> /Reference Block 1/GND_heater
- U3 pad 2: /Reference Block 1/GND_zener -> /Reference Block 6/GND_zener
- U3 pad 4: /Reference Block 1/GND_heater -> /Reference Block 6/GND_heater
- U4 pad 2: /Reference Block 1/GND_zener -> /Reference Block 6/GND_zener
- U4 pad 4: /Reference Block 1/GND_heater -> /Reference Block 6/GND_heater
- U5 pad 2: /Reference Block 5/GND_zener -> /Reference Block 1/GND_zener
- U5 pad 4: /Reference Block 5/GND_heater -> /Reference Block 1/GND_heater
- U6 pad 2: /Reference Block 5/GND_zener -> /Reference Block 1/GND_zener
- U6 pad 4: /Reference Block 5/GND_heater -> /Reference Block 1/GND_heater
- U7 pad 2: /Reference Block 1/GND_zener -> /Reference Block 6/GND_zener
- U7 pad 4: /Reference Block 1/GND_heater -> /Reference Block 6/GND_heater
- U8 pad 2: /Reference Block 1/GND_zener -> /Reference Block 6/GND_zener
- U8 pad 4: /Reference Block 1/GND_heater -> /Reference Block 6/GND_heater
Routing:
- net /Reference Block 5/GND_heater: track 88.0 -> 0.00 mm, vias 2 -> 0
- net /Reference Block 6/GND_heater: track 0.00 -> 87.7 mm, vias 0 -> 2
- net /Reference Block 6/GND_zener: track 0.00 -> 66.4 mm, vias 0 -> 1
- net /Reference Block 5/GND_zener: track 62.8 -> 0.00 mm, vias 1 -> 0
- net /Reference Block 1/GND_zener: track 66.4 -> 62.8 mm
