File: reference_quad_block.kicad_sch (KiCad schematic)
At the start: 3 parts, among them U1 OPA4202

Commit message: Updated references to follow geographical rules
Parts:
- renumbered C1 to C41, NT25 to NT19, U1 to U22
Changed lines of the file:
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@@
 		(on_board yes)
 		(dnp no)
-		(property "Reference" "U1"
+		(property "Reference" "U22"
 			(at 77.47 90.17 0)
 			(effects
@@
 			(project "lm399_burnin_board"
 				(path "/6284122b-79c3-4e04-925e-3d32cc3ec077/00000000-0000-0000-0000-000061945b55"
-					(reference "U1")
+					(reference "U22")
 					(unit 5)
 				)
 				(path "/6284122b-79c3-4e04-925e-3d32cc3ec077/00000000-0000-0000-0000-000061977754"
-					(reference "U6")
+					(reference "U25")
 					(unit 5)
 				)
 				(path "/6284122b-79c3-4e04-925e-3d32cc3ec077/00000000-0000-0000-0000-000061977b94"
-					(reference "U11")
+					(reference "U24")
 					(unit 5)
 				)
 				(path "/6284122b-79c3-4e04-925e-3d32cc3ec077/00000000-0000-0000-0000-00006197812a"
-					(reference "U16")
+					(reference "U26")
 					(unit 5)
 				)
 				(path "/6284122b-79c3-4e04-925e-3d32cc3ec077/00000000-0000-0000-0000-00006197beb8"
-					(reference "U21")
+					(reference "U23")
 					(unit 5)
 				)
@@
 		(on_board yes)
 		(dnp no)
-		(property "Reference" "C1"
+		(property "Reference" "C41"
 			(at 60.96 99.06 0)
 			(effects
@@
 			(project "main"
 				(path "/6284122b-79c3-4e04-925e-3d32cc3ec077/00000000-0000-0000-0000-000061945b55"
-					(reference "C1")
+					(reference "C41")
 					(unit 1)
 				)
 				(path "/6284122b-79c3-4e04-925e-3d32cc3ec077/00000000-0000-0000-0000-000061977754"
-					(reference "C22")
+					(reference "C82")
 					(unit 1)
 				)
 				(path "/6284122b-79c3-4e04-925e-3d32cc3ec077/00000000-0000-0000-0000-000061977b94"
+					(reference "C78")
+					(unit 1)
+				)
+				(path "/6284122b-79c3-4e04-925e-3d32cc3ec077/00000000-0000-0000-0000-00006197812a"
+					(reference "C103")
+					(unit 1)
+				)
+				(path "/6284122b-79c3-4e04-925e-3d32cc3ec077/00000000-0000-0000-0000-00006197beb8"
 					(reference "C43")
-					(unit 1)
-				)
-				(path "/6284122b-79c3-4e04-925e-3d32cc3ec077/00000000-0000-0000-0000-00006197812a"
-					(reference "C64")
-					(unit 1)
-				)
-				(path "/6284122b-79c3-4e04-925e-3d32cc3ec077/00000000-0000-0000-0000-00006197beb8"
-					(reference "C85")
 					(unit 1)
 				)
@@
 		(on_board yes)
 		(dnp no)
-		(property "Reference" "NT25"
+		(property "Reference" "NT19"
 			(at 92.71 133.35 0)
 			(effects
@@
 			(project "main"
 				(path "/6284122b-79c3-4e04-925e-3d32cc3ec077/00000000-0000-0000-0000-000061945b55"
-					(reference "NT25")
+					(reference "NT19")
 					(unit 1)
 				)
@@
 				)
 				(path "/6284122b-79c3-4e04-925e-3d32cc3ec077/00000000-0000-0000-0000-000061977b94"
-					(reference "NT21")
+					(reference "NT23")
 					(unit 1)
 				)
 				(path "/6284122b-79c3-4e04-925e-3d32cc3ec077/00000000-0000-0000-0000-00006197812a"
-					(reference "NT22")
+					(reference "NT26")
 					(unit 1)
 				)
 				(path "/6284122b-79c3-4e04-925e-3d32cc3ec077/00000000-0000-0000-0000-00006197beb8"
-					(reference "NT23")
-					(unit 1)
-				)
+					(reference "NT20")
+					(unit 1)
+				)

Commit message: Added RoHS info
Parts:
- C41: RoHS (none) -> Yes; Temperature (none) -> Tstorage = –55 °C to 155 °C
- U22: RoHS (none) -> Yes; Temperature (none) -> Tstorage = –40 °C to 125 °C
Other:
- sheet sheet6194633C renamed Reference 3
- sheet sheet6196039A renamed Reference 1
- sheet sheet619606CA renamed Reference 2
- sheet sheet619609F2 renamed Reference 4
Changed lines of the file:
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@@
+			)
+		)
+		(property "RoHS" "Yes "
+			(at 73.66 100.33 0)
+			(effects
+				(font
+					(size 1.27 1.27)
+				)
+				(hide yes)
+			)
+		)
+		(property "Temperature" "Tstorage = –40 °C to 125 °C"
+			(at 73.66 100.33 0)
+			(effects
+				(font
+					(size 1.27 1.27)
+				)
+				(hide yes)
 			)
 		)
@@
 			)
 		)
+		(property "RoHS" "Yes"
+			(at 57.15 100.33 0)
+			(effects
+				(font
+					(size 1.27 1.27)
+				)
+				(hide yes)
+			)
+		)
+		(property "Temperature" "Tstorage = –55 °C to 155 °C"
+			(at 57.15 100.33 0)
+			(effects
+				(font
+					(size 1.27 1.27)
+				)
+				(hide yes)
+			)
+		)
 		(pin "1"
 		)
@@
 			(color 0 0 0 0.0000)
 		)
-		(property "Sheetname" "sheet6194633C"
+		(property "Sheetname" "Reference 3"
 			(at 49.53 33.5784 0)
 			(effects
@@
 			(color 0 0 0 0.0000)
 		)
-		(property "Sheetname" "sheet6196039A"
+		(property "Sheetname" "Reference 1"
 			(at 104.14 33.5784 0)
 			(effects
@@
 			(color 0 0 0 0.0000)
 		)
-		(property "Sheetname" "sheet619606CA"
+		(property "Sheetname" "Reference 2"
 			(at 158.75 33.5784 0)
 			(effects
@@
 			(color 0 0 0 0.0000)
 		)
-		(property "Sheetname" "sheet619609F2"
+		(property "Sheetname" "Reference 4"
 			(at 213.36 33.5784 0)
 			(effects
